Commit message: Add deterministic CAD→sim router, URDF ingest, STEP draft spec, and cad2sim skill
Three-layer routing (CAD software, export format, simulator):
- cad2urdf/routes.py + route.py: pick the front end (onshape-to-robot,
  Onshape URDF export, sw2robot, ACDC4Robot, creo2urdf, or STEP) and the
  per-simulator finish, then compile and validate.
- cad2urdf/ingest.py: any exporter URDF into the IR (rotated frames,
  package:// paths, Y-up exports via root_rpy, massless links, mimic).
- cad2urdf/draft.py: deterministic spec for mate-less STEP (touching parts
  form a link, clearance fits are joints, press fits are fixed); recovers
  arm4's 7 links and 6 joint types.
- IR now carries link rotations; URDF/MJCF writers handle fixed,
  continuous and floating-base robots and floor massless MuJoCo bodies.
- collision "auto" mode (per-part primitive / hull / CoACD) is the default.
- validate.py is robot-agnostic and checks ManiSkill on CPU and GPU.
- CoACD is imported lazily: loading it before OpenCascade crashed STEP import.
- cad2sim skill for Claude Code and Codex covers the judgment calls.

Sample CAD fixes: the shoulder pin no longer touches the motor face and the
elbow motor is mounted on the forearm, so the geometry rules group parts
correctly. arm4 outputs, figures and doc numbers regenerated.

Co-Authored-By: Claude Opus 5.5 <noreply@anthropic.com>

File: examples/arm4/output/arm4.urdf (robot description, URDF)
Before this commit: robot arm4, 7 links, 6 joints
Links:
- link forearm: mass 0.350529 -> 0.646467; geometry collision box size=0.03 0.006 0.235; collision box size=0.03 0.006 0.235
- link upper_arm: mass 1.07731 -> 0.77782; geometry collision mesh filename=meshes/collision/upper_arm_0.stl; collision mesh filename=meshes/collision/upper_arm_1.stl

File: examples/arm4/output/gazebo/arm4.gazebo.urdf (robot description, URDF)
Before this commit: robot arm4, 8 links, 7 joints
Links:
- link forearm: mass 0.350529 -> 0.646467; geometry collision box size=0.03 0.006 0.235; collision box size=0.03 0.006 0.235
- link upper_arm: mass 1.07731 -> 0.77782; geometry collision mesh filename=package://arm4_description/meshes/collision/upper_arm_0.stl; collision mesh filename=package://arm4_description/meshes/collision/upper_arm_1.stl
